File: atmega2560/atmega2560.kicad_pcb (KiCad board)
At the start: 2 copper layers, 0 parts

Commit message: Working on digital I/O pins.
Parts:
- added C1: 10uF 25V, Wickerlib:RLC-1210-SMD, F.Cu at (71.9, 76.9)
- added C10: 100nF, Wickerlib:RLC-0603-SMD, F.Cu at (111.0, 52.8)
- added C2: 100nF, Wickerlib:RLC-0603-SMD, F.Cu at (101.1, 98.2)
- added C3: 10uF 25V, Wickerlib:RLC-1210-SMD, F.Cu at (79.6, 84.0)
- added C4: 22pF, Wickerlib:RLC-0603-SMD, F.Cu at (106.8, 92.6)
- added C5: 22pF, Wickerlib:RLC-0603-SMD, F.Cu at (117.1, 92.2)
- added C6: 100nF, Wickerlib:RLC-0603-SMD, F.Cu at (108.8, 68.3)
- added C7: 100nF, Wickerlib:RLC-0603-SMD, F.Cu at (110.8, 61.5)
- added C8: 100nF, Wickerlib:RLC-0603-SMD, F.Cu at (113.8, 65.3)
- added C9: 100nF, Wickerlib:RLC-0603-SMD, F.Cu at (111.2, 57.2)
- added D1: 14V, Wickerlib:DIODE-SMA, F.Cu at (61.5, 69.6)
- added D2: 20V 1A, Wickerlib:DIODE-SMA, F.Cu at (68.7, 67.8)
- added D3: 20V 1A, Wickerlib:DIODE-SMA, F.Cu at (79.2, 91.2)
- added F1: 1.1A 25V, Wickerlib:RLC-1812-SMD, F.Cu at (68.2, 72.6)
- added J1: INPUT, Wickerlib:CONN-ONSHORE-SCREW-GREEN-2PIN-TH, F.Cu at (55.7, 68.1)
- added J2: FTDI, Wickerlib:CONN-HEADER-STRAIGHT-P2.54MM-1x06, F.Cu at (99.1, 66.1)
- added J3: ISP-2560, Wickerlib:CONN-HEADER-STRAIGHT-P2.54MM-2x03, F.Cu at (92.2, 74.9)
- added LED1: AMBER, Wickerlib:LED-0603-SMD, F.Cu at (143.9, 53.0)
- added R1: 1K, Wickerlib:RLC-0603-SMD, F.Cu at (139.9, 53.3)
- added R2: 10K, Wickerlib:RLC-0805-SMD, F.Cu at (101.4, 94.0)
- added S1: RESET, Wickerlib:SWITCH-OMRON-MOMENTARY-SMD-B3U-1000P, F.Cu at (100.9, 104.3)
- added U1: NCP1117-5V, Wickerlib:DPAK, F.Cu at (71.9, 82.5)
- added U2: ATMEGA2560, Wickerlib:TQFP-100-14x14MM-P0.5MM, F.Cu at (113.1, 79.1)
- added X1: 16MHz 18pF, Wickerlib:CRYSTAL-CTS-4SMD, F.Cu at (112.2, 92.2)
