File: atmega2560/atmega2560.kicad_pcb (KiCad board)
At the start: 2 copper layers, 0 parts

Commit message: lots of pin adds to atmega2560
Parts:
- added C1: 10uF 25V, Wickerlib:RLC-1210-SMD, F.Cu at (140.1, 107.1)
- added C10: 100nF, Wickerlib:RLC-0603-SMD, F.Cu at (182.0, 92.2)
- added C2: 100nF, Wickerlib:RLC-0603-SMD, F.Cu at (148.8, 95.4)
- added C3: 10uF 25V, Wickerlib:RLC-1210-SMD, F.Cu at (127.6, 95.6)
- added C4: 22pF, Wickerlib:RLC-0603-SMD, F.Cu at (170.9, 115.9)
- added C5: 22pF, Wickerlib:RLC-0603-SMD, F.Cu at (180.1, 115.3)
- added C6: 100nF, Wickerlib:RLC-0603-SMD, F.Cu at (172.5, 92.3)
- added C7: 100nF, Wickerlib:RLC-0603-SMD, F.Cu at (187.7, 102.9)
- added C8: 100nF, Wickerlib:RLC-0603-SMD, F.Cu at (173.7, 111.9)
- added C9: 100nF, Wickerlib:RLC-0603-SMD, F.Cu at (167.7, 100.8)
- added D1: 14V, Wickerlib:DIODE-SMA, F.Cu at (132.9, 113.8)
- added D2: 20V 1A, Wickerlib:DIODE-SMA, F.Cu at (137.5, 113.7)
- added D3: 20V 1A, Wickerlib:DIODE-SMA, F.Cu at (132.8, 93.7)
- added F1: 1.1A 25V, Wickerlib:RLC-1812-SMD, F.Cu at (142.0, 114.3)
- added J1: INPUT, Wickerlib:CONN-ONSHORE-SCREW-GREEN-2PIN-TH, F.Cu at (125.8, 112.9)
- added J2: FTDI, Wickerlib:CONN-HEADER-STRAIGHT-P2.54MM-1x06, F.Cu at (152.5, 99.0)
- added J3: ISP-2560, Wickerlib:CONN-HEADER-STRAIGHT-P2.54MM-2x03, F.Cu at (144.8, 109.2)
- added J4: ANALOG PINS, Wickerlib:CONN-HEADER-STRAIGHT-P2.54MM-1x16, F.Cu at (157.5, 85.1)
- added J5: HEADER-FEMALE-16POS-TH-1x16-P0.1IN, Wickerlib:CONN-HEADER-STRAIGHT-P2.54MM-1x16, F.Cu at (157.5, 123.2)
- added J6: HEADER-FEMALE-16POS-TH-1x16-P0.1IN, Wickerlib:CONN-HEADER-STRAIGHT-P2.54MM-1x16, F.Cu at (200.7, 85.1)
- added J7: I/O, Wickerlib:CONN-HEADER-STRAIGHT-P2.54MM-1x14, F.Cu at (119.4, 123.2)
- added J8: BARREL JACK, Wickerlib:CONN-BARREL-JACK-2.5x5.5MM-TH, F.Cu at (132.1, 102.8)
- added J9: HEADER-FEMALE-7POS-TH-1x07-P0.1IN, Wickerlib:CONN-HEADER-STRAIGHT-P2.54MM-1x07, F.Cu at (156.2, 97.8)
- added JP1: JUMP, Wickerlib:CONN-HEADER-STRAIGHT-P2.54MM-1x02, F.Cu at (162.3, 93.3)
- added R2: 10K, Wickerlib:RLC-0805-SMD, F.Cu at (160.8, 105.8)
- added S1: RESET, Wickerlib:SWITCH-OMRON-MOMENTARY-SMD-B3U-1000P, F.Cu at (160.8, 113.0)
- added U1: NCP1117-5V, Wickerlib:DPAK, F.Cu at (140.1, 102.7)
- added U2: ATMEGA2560, Wickerlib:TQFP-100-14x14MM-P0.5MM, F.Cu at (177.8, 102.3)
- added X1: 16MHz 18pF, Wickerlib:CRYSTAL-CTS-4SMD, F.Cu at (175.5, 115.8)
Routing:
- net Net-(J4-Pad1): track 0.00 -> 41.6 mm, vias 0 -> 1
- net GND: track 0.00 -> 15.7 mm
- net Net-(C4-Pad1): track 0.00 -> 10.4 mm
- net Net-(C5-Pad1): track 0.00 -> 7.95 mm
- net +5V: track 0.00 -> 5.07 mm
- net /AREF: track 0.00 -> 2.58 mm
- added copper zone on B.Cu, net GND
- added copper zone on F.Cu, net GND
Other:
- board outline added: 86.4 x 43.2 mm
- net class Default: clearance 0.254 -> 0.2032
- rule trace_clearance: 0.1524 -> 0.2032
- board text added: "5V"
- board text added: "AREF"
