File: atmega2560/atmega2560.sch (KiCad schematic (older format))
At the start: 24 parts, among them J1 INPUT, J2 FTDI, J3 ISP-2560, U1 NCP1117-5V, U2 ATMEGA2560, X1 16MHz 18pF

Commit message: Working on digital I/O pins.
Parts:
- removed U2: ATMEGA2560, Wickerlib:TQFP-100-14x14MM-P0.5MM, symbol IC-MCU-ATMEGA2560-SIMPLE
- added U2: ATMEGA2560, Wickerlib:TQFP-100-14x14MM-P0.5MM, symbol IC-MCU-ATMEGA2560-CUSTOM4
- renumbered C2 to C1, C1 to C2, C5 to C3, C3 to C4, C4 to C5, R2 to R1, R1 to R2
Connections:
- net +5V: now also U2.10 (VCC), U2.100 (AVCC), U2.31 (VCC), U2.61 (VCC), U2.80 (VCC), U2.98 (AREF); no longer D3.1 (K)
- net FTDI_RXIN: now also U2.3 ((TXD0)PE1)
- net FTDI_TXOUT: now also U2.2 ((PCINT8/RXD0)PE0)
- net GND: now also U2.11 (GND), U2.32 (GND), U2.62 (GND), U2.81 (GND), U2.99 (GND)
- net MISO: now also U2.22 ((PCINT3/MISO)PB3)
- net MOSI: now also U2.21 ((PCINT2/MOSI)PB2)
- net SCK: now also U2.20 ((PCINT1/SCK)PB1)
- net ~RESET: now also U2.30 (~RESET)
- net at C4.1, X1.1 (EN): now also U2.33 (XTAL2)
- net at C5.1, X1.3 (OUT): now also U2.34 (XTAL1)
Other:
- note removed: "NEED TO ADD BREAKOUT PINS\n"
- moved on the sheet: C1, C10, C2, C3, C4, C5, C6, C7, C8, C9, D1, D2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
