File: atmega2560/atmega2560.sch (KiCad schematic (older format))
At the start: 0 parts

Commit message: lots of pin adds to atmega2560
Parts:
- added C1, C3: 10uF 25V, Wickerlib:RLC-1210-SMD, symbol CAP-CER-10UF-25V-X7R-1210
- added C10, C2, C6, C7, C8, C9: 100nF, Wickerlib:RLC-0603-SMD, symbol CAP-CER-0.1UF-100V-X7R-0603
- added C4, C5: 22pF, Wickerlib:RLC-0603-SMD, symbol CAP-CER-22PF-100V-C0G-NP0-0603
- added D1: 14V, Wickerlib:DIODE-SMA, symbol DIODE-TVS-SMAJ14A-13-F-SMA
- added D2, D3: 20V 1A, Wickerlib:DIODE-SMA, symbol DIODE-SCHOTTKY-20V-1A-SS12-SMA
- added F1: 1.1A 25V, Wickerlib:RLC-1812-SMD, symbol FUSE-RESET-1.1A-25V-MF-MSMF
- added J1: INPUT, Wickerlib:CONN-ONSHORE-SCREW-GREEN-2PIN-TH, symbol CONN-TERM-SCREW-GREEN-2.54MM-2POS-TH
- added J2: FTDI, Wickerlib:CONN-HEADER-STRAIGHT-P2.54MM-1x06, symbol HEADER-MALE-6POS-TH-1x06-P0.1IN
- added J3: ISP-2560, Wickerlib:CONN-HEADER-STRAIGHT-P2.54MM-2x03, symbol HEADER-MALE-6POS-TH-2x3-P0.1IN
- added J4: ANALOG PINS, Wickerlib:CONN-HEADER-STRAIGHT-P2.54MM-1x16, symbol HEADER-FEMALE-16POS-TH-1x16-P0.1IN
- added J8: BARREL JACK, Wickerlib:CONN-BARREL-JACK-2.5x5.5MM-TH, symbol CONN-PWR-JACK-2.0X6.5MM-HIGH-CUR
- added JP1: JUMP, Wickerlib:CONN-HEADER-STRAIGHT-P2.54MM-1x02, symbol SHUNT-JUMPER-2PIN-P0.1IN
- added R2: 10K, Wickerlib:RLC-0805-SMD, symbol RES-10K-5%-1/8W-0805
- added S1: RESET, Wickerlib:SWITCH-OMRON-MOMENTARY-SMD-B3U-1000P, symbol SWITCH-TACTILE-SPST-NO-0.05A-12V
- added U1: NCP1117-5V, Wickerlib:DPAK, symbol IC-REG-LDO-5V-1.1A-NCP1117-5V-DPAK
- added U2: ATMEGA2560, Wickerlib:TQFP-100-14x14MM-P0.5MM, symbol IC-MCU-ATMEGA2560-CUSTOM4
- added X1: 16MHz 18pF, Wickerlib:CRYSTAL-CTS-4SMD, symbol CRYSTAL-16MHZ-18PF-40OHM-CTS-4SMD
Connections:
- new net: C4.1, U2.33 (XTAL2), X1.1 (EN)
- new net: C5.1, U2.34 (XTAL1), X1.3 (OUT)
- new net: C3.1, D3.2 (A), U1.2 (OUT)
- new net: D2.1 (K), F1.2
- new net: J4.1 (P1), U2.97 ((ADC0)PF0)
- new net: J4.10 (P10), U2.88 (PK1(ADC9/PCINT17))
- new net: J4.11 (P11), U2.87 (PK2(ADC10/PCINT18))
- new net: J4.12 (P12), U2.86 (PK3(ADC11/PCINT19))
- new net: J4.13 (P13), U2.85 (PK4(ADC12/PCINT20))
- new net: J4.14 (P14), U2.84 (PK5(ADC13/PCINT21))
- new net: J4.15 (P15), U2.83 (PK6(ADC14/PCINT22))
- new net: J4.16 (P16), U2.82 (PK7(ADC15/PCINT23))
- new net: J4.2 (P2), U2.96 ((ADC1)PF1)
- new net: J4.3 (P3), U2.95 ((ADC2)PF2)
- new net: J4.4 (P4), U2.94 ((ADC3)PF3)
- new net: J4.5 (P5), U2.93 ((TCK/ADC4)PF4)
- new net: J4.6 (P6), U2.92 ((TMS/ADC5)PF5)
- new net: J4.7 (P7), U2.91 ((TD0/ADC6)PF6)
- new net: J4.8 (P8), U2.90 ((TDI/ADC7)PF7)
- new net: J4.9 (P9), U2.89 (PK0(ADC8/PCINT16))
- new net +12V: C1.1, F1.1, U1.3 (IN)
- new net +5V: C10.1, C7.1, C8.1, C9.1, D3.1 (K), J2.4 (P4), J3.2 (P2), JP1.2, R2.1, U2.10 (VCC), U2.100 (AVCC), U2.31 (VCC), U2.61 (VCC), U2.80 (VCC)
- new net AREF: C6.1, JP1.1, U2.98 (AREF)
- new net FTDI_RESET: C2.2, J2.1 (P1)
- new net FTDI_RXIN: J2.3 (P3), U2.3 ((TXD0)PE1)
- new net FTDI_TXOUT: J2.2 (P2), U2.2 ((PCINT8/RXD0)PE0)
- new net GND: C1.2, C10.2, C3.2, C4.2, C5.2, C6.2, C7.2, C8.2, C9.2, D1.2, J1.2 (P2), J2.6 (P6), J3.6 (P6), J8.2, J8.3, S1.1, U1.1 (GND), U2.11 (GND), U2.32 (GND), U2.62 (GND), U2.81 (GND), U2.99 (GND), X1.2 (GND), X1.4 (GND)
- new net MISO: J3.1 (P1), U2.22 ((PCINT3/MISO)PB3)
- new net MOSI: J3.4 (P4), U2.21 ((PCINT2/MOSI)PB2)
- new net SCK: J3.3 (P3), U2.20 ((PCINT1/SCK)PB1)
- new net VIN: D1.1, D2.2 (A), J1.1 (P1), J8.1
- new net ~RESET: C2.1, J3.5 (P5), R2.2, S1.2, U2.30 (~RESET)
- no-connect marks 0 -> 1
Other:
- note added: "Analog\nReference"
- note added: "ICSP\nProgrammer"
- note added: "MAIN INPUT POWER\n-----------\n12V 1A RATING\n"
- note added: "Microcontroller \nInput Voltage"
- note added: "To FTDI\nProgrammer"
