File: usb-breakout/usb-breakout.sch (KiCad schematic (older format))
At the start: 9 parts, among them J1 USB-MICRO, J2 TO MICROCONTROLLER, SW1 RESET

Commit message: USB for safekeeping. Atmega328 v1.2 release.
Parts:
- C1: value 1uF -> 1uf; footprint CAP-5MM-RAD -> Wickerlib:CAP-DISC-D7.5MM-P5MM; Package C_Disc_D7.5_P5 -> (none); Verified Not Verified -> (none)
- D1, D2: Package Diode_DO-41 -> (none); Verified Not Verified -> (none)
- J1: footprint Wickerlib:CONN-USB-MICRO-B-AMPHENOL-10118193-0001LF -> USB-10118193; Package USB_Micro-B_10118193_0001LF -> (none); Verified Not Verified -> (none)
- J2: footprint Wickerlib:CONN-HEADER-STRAIGHT-P2.54MM-1x05 -> CONN-1x05-2.54MM-TH; Package Pin_Header_Straight_1x05 -> (none); Verified Not Verified -> (none)
- R1, R2, R3: Verified Not Verified -> (none)
- SW1: Package SW-B3F-10XX -> (none); Verified Not Verified -> (none)
Connections:
- net DM: now also R2.2; no longer R2.1
- net DP: now also R3.2; no longer R3.1
- net at D1.1 (K), J1.2 (D-), R1.2: now also R2.1; no longer R2.2
- net at D2.1 (K), J1.3 (D+): now also R3.1; no longer R3.2
Other:
- note added: "Breadboard-compatible"
