File: mma7660-sensor-breakout/mma7660-sensor-breakout.sch (KiCad schematic (older format))
At the start: 4 parts, among them J1 HEADER, U1 MMA7660-DFN10

Commit message: Release v1.1 MMA7660 breakout.
Parts:
- added R1, R2: 1K, Wickerlib:RLC-0603-SMD, symbol RES-1K-1%-1/10W-0603
- C1, C2: footprint Wickerlib:RLC-0805-SMD -> Wickerlib:RLC-0805; Package 0805 -> (none); Verified Not Verified -> (none)
- U1: value MMA7660-DFN10 -> IC-MMA7660-DFN10; Package DFN-10-1EP_3x3mm_Pitch0.5mm -> (none); Verified Not Verified -> (none)
Connections:
- net +3V3: now also R1.1, R2.1
- net INT: now reaches J1.2 (P2), U1.5 (~INT)
- net SCL: now reaches J1.4 (P4), U1.6 (SCL)
- net SCL: now also R2.2
- net SDA: now reaches J1.3 (P3), U1.7 (SDA)
- net SDA: now also R1.2
Other:
- note added: "MMA7660 3-axis Accelerometer Sensor Breakout v1.1\n---------------------------------\nAdded onboard I2C pullup resistors.\nC1 and C2 are 0805 package for easier hand soldering.\nThe accelerometer is not 5V-tolerant. You must supply 3.3V."
- note removed: "MMA7660 3-axis Accelerometer Sensor Breakout v1.0\n---------------------------------\nThere are no onboard I2C pullup lines.\nC1 and C2 are 0805 package for easier hand soldering.\nThe accelerometer is not 5V-tolerant. You must supply 3.3V."
- moved on the sheet: J1
