File: sd-micro-pushpull-0475710001-breakout/sd-micro-pushpull-0475710001-breakout.sch (KiCad schematic (older format))
At the start: 0 parts

Commit message: Release v1.0 MicroSD Push-Pull Breakout
Parts:
- added C1, C4: 1uF, Wickerlib:RLC-0603-SMD, symbol CAP-CER-1UF-25V-X7R-0603
- added C2, C3: 0.1uF, Wickerlib:RLC-0603-SMD, symbol CAP-CER-0.1UF-100V-X7R-0603
- added J1: BREAKOUT, Wickerlib:CONN-HEADER-STRAIGHT-P2.54MM-1x06, symbol HEADER-MALE-6POS-TH-1x06-P0.1IN
- added J2: CONN-MICRO-SD-CARD-PUSH-PULL, Wickerlib:CONN-SD-MICRO-MOLEX-0475710001, symbol CONN-MICRO-SD-CARD-PUSH-PULL
- added U1: MIC5365 150mA, Wickerlib:SOT-353, symbol IC-REG-LDO-3.3V-0.15A-MIC5365-SOT353
- added U2: TXB0104, Wickerlib:SOIC-14-3.9x8.7MM-P1.27MM, symbol IC-VOLT-LEVEL-TRANSLATOR-TXB0104-SOIC14
Connections:
- new net +3V3: C3.1, C4.1, J2.4 (VCC), U1.5 (VOUT), U2.1 (VCCA), U2.8 (OE)
- new net CLK: J1.3 (P3), U2.12 (B2)
- new net CS: J1.5 (P5), U2.10 (B4)
- new net GND: C1.2, C2.2, C3.2, C4.2, J1.6 (P6), J2.6 (VSS), U1.2 (GND), U2.7 (GND)
- new net MISO: J1.2 (P2), U2.13 (B1)
- new net MOSI: J1.4 (P4), U2.11 (B3)
- new net SD_CLK: J2.5 (SCLK), U2.3 (A2)
- new net SD_CS: J2.2 (CS), U2.5 (A4)
- new net SD_MISO: J2.7 (DATA_OUT), U2.2 (A1)
- new net SD_MOSI: J2.3 (DATA_IN), U2.4 (A3)
- new net VIN: C1.1, C2.1, J1.1 (P1), U1.1 (VIN), U1.3 (STBY), U2.14 (VCCB)
