File: sd-micro-pushpull-0475710001-breakout/sd-micro-pushpull-0475710001-breakout.kicad_pcb (KiCad board)
At the start: 2 copper layers, 0 parts

Commit message: Release v1.0 MicroSD Push-Pull Breakout
Parts:
- added C1: 1uF, Wickerlib:RLC-0603-SMD, F.Cu at (133.1, 106.2)
- added C2: 0.1uF, Wickerlib:RLC-0603-SMD, F.Cu at (130.6, 102.9)
- added C3: 0.1uF, Wickerlib:RLC-0603-SMD, F.Cu at (130.6, 95.2)
- added C4: 1uF, Wickerlib:RLC-0603-SMD, F.Cu at (138.2, 106.2)
- added J1: BREAKOUT, Wickerlib:CONN-HEADER-STRAIGHT-P2.54MM-1x06, F.Cu at (123.7, 106.7)
- added J2: CONN-MICRO-SD-CARD-PUSH-PULL, Wickerlib:CONN-SD-MICRO-MOLEX-0475710001, F.Cu at (140.7, 100.1)
- added U1: MIC5365 150mA, Wickerlib:SOT-353, F.Cu at (135.6, 106.5)
- added U2: TXB0104, Wickerlib:SOIC-14-3.9x8.7MM-P1.27MM, F.Cu at (136.3, 99.1)
Routing:
- net +3V3: track 0.00 -> 28.7 mm, vias 0 -> 2
- net GND: track 0.00 -> 21.8 mm, vias 0 -> 8
- net VIN: track 0.00 -> 19.3 mm
- net /MISO: track 0.00 -> 11.0 mm
- net /CS: track 0.00 -> 10.4 mm
- net /CLK: track 0.00 -> 10.4 mm
- net /MOSI: track 0.00 -> 9.91 mm
- net /SD_MISO: track 0.00 -> 3.56 mm
- net /SD_MOSI: track 0.00 -> 3.24 mm
- net /SD_CLK: track 0.00 -> 3.17 mm
- net /SD_CS: track 0.00 -> 3.17 mm
- added copper zone on B.Cu, net GND
- added copper zone on F.Cu, net GND
Other:
- board outline added: 24.9 x 16.3 mm
- rule trace_clearance: 0.1524 -> 0.254
- board text added: "CLK"
- board text added: "CS"
- board text added: "GND"
- board text added: "MISO"
- board text added: "MOSI"
- board text added: "MicroSD Card Breakout"
- board text added: "Narrow Micro SD Card Breakout"
- board text added: "SD Connector: Molex P/N 0475710001 VIN can be 5V or 3.3V wickerbox.net"
- board text added: "VIN"
- board text added: "v1.0 1/4/17"

Commit message: Ran updated docs output.
Other:
- board text removed: "Narrow Micro SD Card Breakout"
- board text removed: "v1.0 1/4/17"
Changed lines of the file:
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@@
-(kicad_pcb (version 4) (host pcbnew 4.0.4+e1-6308~48~ubuntu16.04.1-stable)
+(kicad_pcb (version 4) (host pcbnew 4.0.5-e0-6337~49~ubuntu16.04.1)
   (general
     (links 25)
@@
     (area 104.572999 74.854999 178.510001 123.265001)
     (thickness 1.6)
-    (drawings 43)
+    (drawings 41)
     (tracks 88)
     (zones 0)
@@
       (net 1 VIN))
   )
+  (gr_arc (start 145.034 93.98) (end 145.034 92.202) (angle 90) (layer F.Fab) (width 0.1524))
+  (gr_line (start 121.92 93.98) (end 121.92 106.68) (layer F.Fab) (width 0.1524))
+  (gr_arc (start 123.698 106.68) (end 123.698 108.458) (angle 90) (layer F.Fab) (width 0.1524))
+  (gr_line (start 145.034 108.458) (end 123.698 108.458) (layer F.Fab) (width 0.1524))
   (gr_text "SD Connector:\nMolex P/N 0475710001\n\nVIN can be 5V or 3.3V\n\nwickerbox.net" (at 135.128 101.854) (layer B.SilkS)
     (effects (font (size 1.016 1.016) (thickness 0.1524)) (justify mirror))
   )
-  (gr_text "v1.0                    1/4/17" (at 134.62 110.236) (layer F.Fab)
-    (effects (font (size 1.016 1.016) (thickness 0.1524)))
-  )
   (gr_text "MicroSD Card Breakout" (at 135.636 94.234) (layer B.SilkS)
     (effects (font (size 1.016 1.016) (thickness 0.1524)) (justify mirror))
-  )
-  (gr_text "Narrow Micro SD Card Breakout" (at 134.62 90.932) (layer F.Fab)
-    (effects (font (size 1.016 1.016) (thickness 0.1524)))
   )
   (gr_line (start 121.92 93.98) (end 121.92 106.68) (layer Edge.Cuts) (width 0.1524))
@@
   (gr_line (start 123.698 92.202) (end 145.034 92.202) (layer Edge.Cuts) (width 0.1524))
   (gr_arc (start 123.698 93.98) (end 121.92 93.98) (angle 90) (layer Edge.Cuts) (width 0.1524))
-  (gr_line (start 121.92 93.98) (end 121.92 106.68) (layer F.Fab) (width 0.1524))
   (gr_line (start 146.812 93.98) (end 146.812 106.68) (layer F.Fab) (width 0.1524))
-  (gr_arc (start 123.698 106.68) (end 123.698 108.458) (angle 90) (layer F.Fab) (width 0.1524))
-  (gr_line (start 145.034 108.458) (end 123.698 108.458) (layer F.Fab) (width 0.1524))
   (gr_arc (start 145.034 106.68) (end 146.812 106.68) (angle 90) (layer F.Fab) (width 0.1524))
-  (gr_arc (start 145.034 93.98) (end 145.034 92.202) (angle 90) (layer F.Fab) (width 0.1524))
   (gr_line (start 123.698 92.202) (end 145.034 92.202) (layer F.Fab) (width 0.1524))
   (gr_arc (start 123.698 93.98) (end 121.92 93.98) (angle 90) (layer F.Fab) (width 0.1524))
