File: sd-full-2041021-4-breakout/sd-full-2041021-4-breakout.kicad_pcb (KiCad board)
At the start: 2 copper layers, 0 parts

Commit message: Update docs. Release full SD breakout v1.0
Parts:
- added C1: 1uF, Wickerlib:RLC-0603-SMD, F.Cu at (107.4, 86.6)
- added C2: 0.1uF, Wickerlib:RLC-0603-SMD, F.Cu at (107.7, 81.8)
- added C3: 0.1uF, Wickerlib:RLC-0603-SMD, F.Cu at (107.7, 70.6)
- added C4: 1uF, Wickerlib:RLC-0603-SMD, F.Cu at (112.8, 86.6)
- added J1: BREAKOUT, Wickerlib:CONN-HEADER-STRAIGHT-P2.54MM-1x06, F.Cu at (100.1, 86.4)
- added J2: TE CONN 2041021-4, Wickerlib:CONN-SD-FULL-TECONN-2041021-4, F.Cu at (116.1, 78.2)
- added U1: MIC5365 150mA, Wickerlib:SOT-353, F.Cu at (110.0, 86.7)
- added U2: TXB0104, Wickerlib:SOIC-14-3.9x8.7MM-P1.27MM, F.Cu at (110.1, 76.2)
Routing:
- net +3V3: track 0.00 -> 31.1 mm, vias 0 -> 3
- net VIN: track 0.00 -> 19.0 mm
- net GND: track 0.00 -> 10.9 mm, vias 0 -> 7
- net /MISO: track 0.00 -> 9.47 mm
- net /SD_MISO: track 0.00 -> 9.22 mm
- net /SCLK: track 0.00 -> 8.94 mm
- net /MOSI: track 0.00 -> 8.51 mm
- net /CS: track 0.00 -> 7.89 mm
- net /SD_CS: track 0.00 -> 5.76 mm
- net /SD_SCLK: track 0.00 -> 5.56 mm
- net /SD_MOSI: track 0.00 -> 4.38 mm
- added copper zone on B.Cu, net GND
- added copper zone on F.Cu, net GND
Other:
- board outline added: 44.5 x 29.2 mm
- rule trace_clearance: 0.1524 -> 0.254
- board text added: "1/4/17"
- board text added: "CS"
- board text added: "Full-size SD Card Breakout SD Connector: TE CONN P/N 2041021-4 VIN can be 5V or 3.3V wickerbox.net"
- board text added: "GND"
- board text added: "MISO"
- board text added: "MOSI"
- board text added: "SCLK"
- board text added: "SD Card Breakout Board v1.0"
- board text added: "VIN"
