File: neopixel-ws2812b-breakout/neopixel-ws2812b-breakout.sch (KiCad schematic (older format))
At the start: 4 parts, among them J1 INPUT, J2 OUTPUT

Commit message: Release Neopixel v1.1. Fixed swapped pads.
Other:
- note added: "Strongly recommended to place \na 100nF capacitor between VCC\nand GND between micro and pixels."
Changed lines of the file:
@@
 Title "Neopixel WS2812B Breakout Board"
 Date "1 Sep 2016"
-Rev"v1.0"
-Comp "CERN Open Hardware License v1.2")
-Comment1 "jenner@wickerbox.net")
-Comment2 "http://wickerbox.net")
-Comment3 "Wickerbox Electronics")
+Rev "v1.0"
+Comp "CERN Open Hardware License v1.2"
+Comment1 "jenner@wickerbox.net"
+Comment2 "http://wickerbox.net"
+Comment3 "Wickerbox Electronics"
 Comment4 ""
 $EndDescr
@@
 $EndComp
 $Comp
-L GND #PWR1
+L GND #PWR01
 U 1 1 57C8B8D5
 P 5550 4700
-F 0 "#PWR1" H 5550 4450 50  0001 C CNN
+F 0 "#PWR01" H 5550 4450 50  0001 C CNN
 F 1 "GND" H 5550 4550 50  0000 C CNN
 F 2 "" H 5550 4700 50  0000 C CNN
@@
 Text Notes 4250 4850 0    60   ~ 0
 Add R1 between \nmicrocontroller\ndata pin and \nNeopixel data input to\nprevent voltage spikes.
+Text Notes 4275 3375 0    60   ~ 0
+Strongly recommended to place \na 100nF capacitor between VCC\nand GND between micro and pixels.
 $EndSCHEMATC
