File: avr-programmer/avr-programmer.sch (KiCad schematic (older format))
At the start: 11 parts, among them J1 FTDI, J2 ISP-2560, U1 ATMEGA328, X1 16MHz 18pF

Commit message: Add switch to AVR Programmer v1.1
Parts:
- added C4: 1uF, Wickerlib:RLC-0603-SMD, symbol CAP-CER-1UF-25V-X7R-0603
- added S2: SLIDE, Wickerlib:SWITCH-ESWITCH-SLIDE-TH-EG1218, symbol SWITCH-SLIDE-SPDT-200MA-30V
Connections:
- net GND: now also C4.2
- net ~RESET: now also S2.1; no longer J2.5 (P5)
- net CS_D10: now reaches U1.14 ((PCINT2/OC1B/~SS~)PB2)
- net CS_D10: now also S2.3
- net +5V renamed VIN
- net VIN: now also C4.1
- new net ISP_RST: J2.5 (P5), S2.2
- no-connect marks 18 -> 17
Other:
- note added: "Microcontroller"
- note added: "Note: crystal\ncould be 20MHz"
- note added: "VIN can be any input voltage\nin range accepted by Atmega328"
- moved on the sheet: R1, S1
