File: atmega328/atmega328.sch (KiCad schematic (older format))
At the start: 25 parts, among them J1 INPUT, J2 FTDI, J3 ISP-2560, J4 DIGOUT1, J5 DIGOUT2, U1 NCP1117-5V, U2 ATMEGA328, X1 16MHz 18pF

Commit message: Added Atmega328 v1.1 to fix Tx/Rx and add breakout pins.
Parts:
- removed J4: DIGOUT1, Wickerlib:Pin_Header_Straight_1x10, symbol HEADER-FEMALE-10POS-TH-1x10-P0.1IN
- removed J5: DIGOUT2, Wickerlib:Pin_Header_Straight_1x10, symbol HEADER-FEMALE-10POS-TH-1x10-P0.1IN
- removed R2: 1K, Wickerlib:0603, symbol RES-1K-1%-1/10W-0603
- removed U2: ATMEGA328, Wickerlib:TQFP-32_7x7mm_Pitch0.8mm, symbol IC-MCU-ATMEGA328-TQFP32
- added J4, J5: HEADER-FEMALE-12POS-TH-1x12-P0.1IN, Wickerlib:CONN-HEADER-STRAIGHT-P2.54MM-1x12, symbol HEADER-FEMALE-12POS-TH-1x12-P0.1IN
- added R2: 220, Wickerlib:RLC-0603-SMD, symbol RES-220-5%-1/10W-0603
- added U2: IC-MCU-ATMEGA328-TQFP32-CUSTOM1, Wickerlib:TQFP-32-7x7MM-P0.8MM, symbol IC-MCU-ATMEGA328-TQFP32-CUSTOM1
- C1, C3, C4, C5, C7, C8, C9, LED1: footprint Wickerlib:0603 -> Wickerlib:RLC-0603-SMD
- C2, C6: footprint Wickerlib:1210 -> Wickerlib:RLC-1210-SMD
- D1, D2, D3: footprint Wickerlib:Diode_SMA -> Wickerlib:DIODE-SMA
- F1: footprint Wickerlib:1812 -> Wickerlib:RLC-1812-SMD
- J1: footprint Wickerlib:OSTVN02A150 -> Wickerlib:CONN-ONSHORE-SCREW-GREEN-2PIN-TH
- J2: footprint Wickerlib:Pin_Header_Straight_1x06 -> Wickerlib:CONN-HEADER-STRAIGHT-P2.54MM-1x06
- J3: footprint Wickerlib:Pin_Header_Straight_2x03 -> Wickerlib:CONN-HEADER-STRAIGHT-P2.54MM-2x03
- R1: footprint Wickerlib:0805 -> Wickerlib:RLC-0805-SMD
- S1: footprint Wickerlib:SW-B3U-1000P -> Wickerlib:SWITCH-OMRON-MOMENTARY-SMD-B3U-1000P
Connections:
- net labels added: FTDI_RX/D1_TX, FTDI_TX/D0_RX
- net labels removed: D0, D1, FTDI_RXIN, FTDI_TXOUT
- wire segments 98 -> 106
Other:
- moved on the sheet: LED1

Commit message: New amazing script updated all kinds of stuff.
Parts:
- X1: Description 16MHz ±30ppm Crystal 18pF 40 Ohm 4SMD NOLEAD -> 16MHz 30ppm Crystal 18pF 40 Ohm 4SMD NOLEAD
Changed lines of the file:
@@
 F 7 "Digikey" H 4025 3525 50  0001 C CIN "S1_Name"
 F 8 "CTX1206CT-ND" H 4025 3525 50  0001 C CIN "S1_PN"
-F 9 "16MHz ±30ppm Crystal 18pF 40 Ohm 4SMD NOLEAD" H 4025 3525 50  0001 C CIN "Description"
+F 9 "16MHz 30ppm Crystal 18pF 40 Ohm 4SMD NOLEAD" H 4025 3525 50  0001 C CIN "Description"
 F 10 "Not Verified" H 4025 3525 50  0001 C CIN "Verified"
 	1    4025 3875

Commit message: Created new atmega328 project folder.
Parts:
- removed C1, C5, C7, C8, C9: 100nF, Wickerlib:RLC-0603-SMD, symbol CAP-CER-0.1UF-100V-X7R-0603
- removed C2, C6: 10uF 25V, Wickerlib:RLC-1210-SMD, symbol CAP-CER-10UF-25V-X7R-1210
- removed C3, C4: 22pF, Wickerlib:RLC-0603-SMD, symbol CAP-CER-22PF-100V-C0G-NP0-0603
- removed D1: 14V, Wickerlib:DIODE-SMA, symbol DIODE-TVS-SMAJ14A-13-F-SMA
- removed D2, D3: 20V 1A, Wickerlib:DIODE-SMA, symbol DIODE-SCHOTTKY-20V-1A-SS12-SMA
- removed F1: 1.1A 25V, Wickerlib:RLC-1812-SMD, symbol FUSE-RESET-1.1A-25V-MF-MSMF
- removed J1: INPUT, Wickerlib:CONN-ONSHORE-SCREW-GREEN-2PIN-TH, symbol CONN-TERM-SCREW-GREEN-2.54MM-2POS-TH
- removed J2: FTDI, Wickerlib:CONN-HEADER-STRAIGHT-P2.54MM-1x06, symbol HEADER-MALE-6POS-TH-1x06-P0.1IN
- removed J3: ISP-2560, Wickerlib:CONN-HEADER-STRAIGHT-P2.54MM-2x03, symbol HEADER-MALE-6POS-TH-2x3-P0.1IN
- removed J4, J5: HEADER-FEMALE-12POS-TH-1x12-P0.1IN, Wickerlib:CONN-HEADER-STRAIGHT-P2.54MM-1x12, symbol HEADER-FEMALE-12POS-TH-1x12-P0.1IN
- removed LED1: AMBER, Wickerlib:RLC-0603-SMD, symbol LED-AMBER-0603-SMT-L296-Q2R2
- removed R1: 10K, Wickerlib:RLC-0805-SMD, symbol RES-10K-5%-1/8W-0805
- removed R2: 220, Wickerlib:RLC-0603-SMD, symbol RES-220-5%-1/10W-0603
- removed S1: RESET, Wickerlib:SWITCH-OMRON-MOMENTARY-SMD-B3U-1000P, symbol SWITCH-TACTILE-SPST-NO-0.05A-12V
- removed U1: NCP1117-5V, Wickerlib:DPAK, symbol IC-REG-LDO-5V-1.1A-NCP1117-5V-DPAK
- removed U2: IC-MCU-ATMEGA328-TQFP32-CUSTOM1, Wickerlib:TQFP-32-7x7MM-P0.8MM, symbol IC-MCU-ATMEGA328-TQFP32-CUSTOM1
- removed X1: 16MHz 18pF, Wickerlib:CRYSTAL-CTS-4SMD, symbol CRYSTAL-16MHZ-18PF-40OHM-CTS-4SMD
Connections:
- net labels removed: +12V, +5V, A0, A1, A2, A3, A4, A5, A6(*), A7(*), AREF, D10, D11, D12, D13, D2, D3, D4, D5, D6, D7, D8, D9, FTDI_RESET, FTDI_RX/D1_TX, FTDI_TX/D0_RX, GND, MISO, MOSI, SCK, VIN, ~RESET
- wire segments 106 -> 0
- no-connect marks 1 -> 0
Other:
- note removed: "* ADC6 and ADC7 can only\nbe used as analog inputs"
- note removed: "Analog\nReference"
- note removed: "Heartbeat"
- note removed: "ICSP\nProgrammer"
- note removed: "MAIN INPUT POWER\n-----------\nSCREW TERMINAL\n12V 1A RATING\n"
- note removed: "To FTDI\nProgrammer"

Commit message: Converted atmega328 to new project format.
Parts:
- added C1, C5, C7, C8, C9: 100nF, Wickerlib:RLC-0603-SMD, symbol CAP-CER-0.1UF-100V-X7R-0603
- added C2, C6: 10uF 25V, Wickerlib:RLC-1210-SMD, symbol CAP-CER-10UF-25V-X7R-1210
- added C3, C4: 22pF, Wickerlib:RLC-0603-SMD, symbol CAP-CER-22PF-100V-C0G-NP0-0603
- added D1: 14V, Wickerlib:DIODE-SMA, symbol DIODE-TVS-SMAJ14A-13-F-SMA
- added D2, D3: 20V 1A, Wickerlib:DIODE-SMA, symbol DIODE-SCHOTTKY-20V-1A-SS12-SMA-RESCUE-atmega328
- added F1: 1.1A 25V, Wickerlib:RLC-1812-SMD, symbol FUSE-RESET-1.1A-25V-MF-MSMF
- added J1: INPUT, Wickerlib:CONN-ONSHORE-SCREW-GREEN-2PIN-TH, symbol CONN-TERM-SCREW-GREEN-2.54MM-2POS-TH
- added J2: FTDI, Wickerlib:CONN-HEADER-STRAIGHT-P2.54MM-1x06, symbol HEADER-MALE-6POS-TH-1x06-P0.1IN
- added J3: ISP-2560, Wickerlib:CONN-HEADER-STRAIGHT-P2.54MM-2x03, symbol HEADER-MALE-6POS-TH-2x3-P0.1IN
- added J4, J5: HEADER-FEMALE-12POS-TH-1x12-P0.1IN, Wickerlib:CONN-HEADER-STRAIGHT-P2.54MM-1x12, symbol HEADER-FEMALE-12POS-TH-1x12-P0.1IN
- added J?: CONN-MICRO-SD-CARD-PUSH-PULL, Wickerlib:CONN-SD-MICRO-MOLEX-0475710001, symbol CONN-MICRO-SD-CARD-PUSH-PULL
- added LED1: AMBER, Wickerlib:RLC-0603-SMD, symbol LED-AMBER-0603-SMT-L296-Q2R2
- added R1: 10K, Wickerlib:RLC-0805-SMD, symbol RES-10K-5%-1/8W-0805
- added R2: 220, Wickerlib:RLC-0603-SMD, symbol RES-220-5%-1/10W-0603
- added S1: RESET, Wickerlib:SWITCH-OMRON-MOMENTARY-SMD-B3U-1000P, symbol SWITCH-TACTILE-SPST-NO-0.05A-12V
- added U1: NCP1117-5V, Wickerlib:DPAK, symbol IC-REG-LDO-5V-1.1A-NCP1117-5V-DPAK
- added U2: IC-MCU-ATMEGA328-TQFP32-CUSTOM1, Wickerlib:TQFP-32-7x7MM-P0.8MM, symbol IC-MCU-ATMEGA328-TQFP32-CUSTOM1
- added X1: 16MHz 18pF, Wickerlib:CRYSTAL-CTS-4SMD, symbol CRYSTAL-16MHZ-18PF-40OHM-CTS-4SMD
Connections:
- net labels added: +12V, +5V, A0, A1, A2, A3, A4, A5, A6(*), A7(*), AREF, D10, D11, D12, D13, D2, D3, D4, D5, D6, D7, D8, D9, FTDI_RESET, FTDI_RX/D1_TX, FTDI_TX/D0_RX, GND, MISO, MOSI, SCK, VIN, ~RESET
- wire segments 0 -> 106
- no-connect marks 0 -> 1
Other:
- note added: "* ADC6 and ADC7 can only\nbe used as analog inputs"
- note added: "Analog\nReference"
- note added: "Heartbeat"
- note added: "ICSP\nProgrammer"
- note added: "MAIN INPUT POWER\n-----------\nSCREW TERMINAL\n12V 1A RATING\n"
- note added: "To FTDI\nProgrammer"

Commit message: Added shunt jumper.
Parts:
- removed D2, D3: 20V 1A, Wickerlib:DIODE-SMA, symbol DIODE-SCHOTTKY-20V-1A-SS12-SMA-RESCUE-atmega328
- removed J?: CONN-MICRO-SD-CARD-PUSH-PULL, Wickerlib:CONN-SD-MICRO-MOLEX-0475710001, symbol CONN-MICRO-SD-CARD-PUSH-PULL
- added D2, D3: 20V 1A, Wickerlib:DIODE-SMA, symbol DIODE-SCHOTTKY-20V-1A-SS12-SMA
- added JP1: JUMP, Wickerlib:CONN-HEADER-STRAIGHT-P2.54MM-1x02, symbol SHUNT-JUMPER-2PIN-P0.1IN
- U2: value IC-MCU-ATMEGA328-TQFP32-CUSTOM1 -> ATMEGA328; Package UNDEFINED -> (none); Verified Not Verified -> (none)
Connections:
- wire segments 106 -> 108
Other:
- note added: "Indicator LED"
- note removed: "Heartbeat"
- moved on the sheet: C5

Commit message: USB for safekeeping. Atmega328 v1.2 release.
Parts:
- X1: Description 16MHz 30ppm Crystal 18pF 40 Ohm 4SMD NOLEAD -> CRYSTAL 16MHz 18pF 40 OHM 4SMD
Changed lines of the file:
@@
 EESchema Schematic File Version 2
 LIBS:wickerlib
+LIBS:atmega328-cache
 EELAYER 25 0
 EELAYER END
@@
 F 7 "Digikey" H 4025 3525 50  0001 C CIN "S1_Name"
 F 8 "CTX1206CT-ND" H 4025 3525 50  0001 C CIN "S1_PN"
-F 9 "16MHz 30ppm Crystal 18pF 40 Ohm 4SMD NOLEAD" H 4025 3525 50  0001 C CIN "Description"
+F 9 "CRYSTAL 16MHz 18pF 40 OHM 4SMD" H 4025 3525 50  0001 C CIN "Description"
 F 10 "Not Verified" H 4025 3525 50  0001 C CIN "Verified"
 	1    4025 3875
