File: fgpmmopa6h-gps-breakout/fgpmmopa6h-gps-breakout.sch (KiCad schematic (older format))
At the start: 15 parts, among them J1 BREAKOUT, U1 MIC5365, U2 FGPMMOPA6H-GPS

Commit message: Release FGPMMOPA6H GPS breakout v1.0
Parts:
- removed J1: BREAKOUT, Wickerlib:CONN-HEADER-STRAIGHT-P2.54MM-1x09, symbol HEADER-MALE-9POS-TH-1x09-P0.1IN
- added J1: BREAKOUT, Wickerlib:CONN-HEADER-STRAIGHT-P2.54MM-1x10, symbol HEADER-MALE-10POS-TH-1x10-P0.1IN
- BAT1: footprint Wickerlib:BATT-HOLDER-STRAP-CR2032-BC-2003 -> Wickerlib:BATT-HOLDER-CR1220-BK-916
Connections:
- net labels added: 3.3V_TX, 5V_TX, ~RESET
- net labels removed: FTDI_RX, FTDI_TX, ~FTDI_RESET, ~GPS_RESET
- wire segments 58 -> 59
- no-connect marks 1 -> 2
Other:
- note added: "1PPS, RTCM, and the FIX \nare 3.3V-level signals and\nmay not be interpreted \ncorrectly by a 5V system."
- note added: "5V FTDI"
- note added: "Based on Adafruit Ultimate GPS Breakout [1]\nand FGPMMOPA6H datasheet [2] reference circuits.\n\n[1] https://www.adafruit.com/products/790\n[2] https://cdn-shop.adafruit.com/datasheets/GlobalTop-FGPMMOPA6H-Datasheet-V0A.pdf"
- note added: "RTCM is not enabled\nby default. Included\nfor completeness."
- note added: "The 5V FTDI cable is for\nif you really just want to\ntalk with the chip over\nRX and TX only."
- note added: "To use with 5V FTDI:\nconnect FTDI cable\nstarting with RESET\n(green) at pin 1.\n\n\nTo use with 3.3V\ncontroller, connect\n to 3.3V, GPS_RX, \n3.3V_TX, and GND."
- note removed: "FTDI-compatible!\n\nPlace FTDI connector \nstarting with RESET\n(green) at pin 1"
- moved on the sheet: AN1, BAT1, C1, C2, C3, C4, LED1, R1, R2, R3, S1, U1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

Commit message: Figuring out Rx/Tx mixup
Parts:
- added J2: 3.3V, Wickerlib:CONN-HEADER-STRAIGHT-P2.54MM-1x01, symbol HEADER-MALE-1POS-TH-1x01
Connections:
- net labels added: 3.3V_RX, 5V_RX
- net labels removed: 5V_TX, GPS_RX, GPS_TX
- wire segments 59 -> 73
Other:
- note added: "FTDI RX\n"
- note added: "FTDI_TX\n"
- moved on the sheet: R1
Changed lines of the file:
@@
 L RES-10K-1%-1/8W-0603 R1
 U 1 1 5874DDA9
-P 4125 2425
-F 0 "R1" H 4175 2475 50  0000 L CNN
-F 1 "10K" H 4175 2375 50  0000 L CNN
-F 2 "Wickerlib:RLC-0603-SMD" H 4125 2075 50  0001 C CIN
-F 3 "http://www.seielect.com/catalog/SEI-RNCP.pdf" H 4125 2425 5   0001 C CNN
-F 4 "RES SMD 10K OHM 1% 1/8W 0603" H 4125 2075 50  0001 C CIN "Description"
-F 5 "Stackpole" H 4125 2075 50  0001 C CIN "MF_Name"
-F 6 "RNCP0603FTD10K0" H 4125 2075 50  0001 C CIN "MF_PN"
-F 7 "Digikey" H 4125 2075 50  0001 C CIN "S1_Name"
-F 8 "RNCP0603FTD10K0CT-ND" H 4125 2075 50  0001 C CIN "S1_PN"
-	1    4125 2425
+P 4425 2575
+F 0 "R1" H 4475 2625 50  0000 L CNN
+F 1 "10K" H 4475 2525 50  0000 L CNN
+F 2 "Wickerlib:RLC-0603-SMD" H 4425 2225 50  0001 C CIN
+F 3 "http://www.seielect.com/catalog/SEI-RNCP.pdf" H 4425 2575 5   0001 C CNN
+F 4 "RES SMD 10K OHM 1% 1/8W 0603" H 4425 2225 50  0001 C CIN "Description"
+F 5 "Stackpole" H 4425 2225 50  0001 C CIN "MF_Name"
+F 6 "RNCP0603FTD10K0" H 4425 2225 50  0001 C CIN "MF_PN"
+F 7 "Digikey" H 4425 2225 50  0001 C CIN "S1_Name"
+F 8 "RNCP0603FTD10K0CT-ND" H 4425 2225 50  0001 C CIN "S1_PN"
+	1    4425 2575
 	1    0    0    -1
 $EndComp
@@
 3D-FIX
 Text Label 6200 3625 0    50   ~ 0
-GPS_RX
+3.3V_RX
 Text Label 6200 3525 0    50   ~ 0
-GPS_TX
+3.3V_TX
 Text Label 6150 3425 0    50   ~ 0
 VBACKUP
@@
 L +3.3V #PWR012
 U 1 1 58752BB1
-P 4125 2325
-F 0 "#PWR012" H 4125 2175 50  0001 C CNN
-F 1 "+3.3V" H 4125 2465 50  0000 C CNN
-F 2 "" H 4125 2325 50  0000 C CNN
-F 3 "" H 4125 2325 50  0000 C CNN
-	1    4125 2325
+P 4425 2475
+F 0 "#PWR012" H 4425 2325 50  0001 C CNN
+F 1 "+3.3V" H 4425 2615 50  0000 C CNN
+F 2 "" H 4425 2475 50  0000 C CNN
+F 3 "" H 4425 2475 50  0000 C CNN
+	1    4425 2475
 	1    0    0    -1
 $EndComp
@@
 NoConn ~ 2375 3125
 Text Label 2625 3625 0    50   ~ 0
-3.3V_TX
-Text Label 2625 2825 0    50   ~ 0
-GPS_RX
-Text Label 2625 2925 0    50   ~ 0
-5V_TX
+3.3V_RX
 $Comp
 L HEADER-MALE-10POS-TH-1x10-P0.1IN J1
@@
 Text Notes 2075 2500 0    50   ~ 0
 5V FTDI
+Text Notes 2625 2825 0    50   ~ 0
+FTDI RX\n
+Text Notes 2625 2925 0    50   ~ 0
+FTDI_TX\n
+Text Label 3000 2925 0    50   ~ 0
+5V_RX
 Connection ~ 8350 4075
 Wire Wire Line
@@
 	8250 3975 8350 3975
 Wire Wire Line
-	8350 3975 8350 4325
+	8350 3975 8350 4075
+Wire Wire Line
+	8350 4075 8350 4175
+Wire Wire Line
+	8350 4175 8350 4275
+Wire Wire Line
+	8350 4275 8350 4325
 Wire Wire Line
 	8250 4275 8350 4275
@@
 	5950 3275 7175 3275
 Wire Wire Line
-	7100 1400 7100 3175
+	7100 1400 7100 1575
+Wire Wire Line
+	7100 1575 7100 2075
+Wire Wire Line
+	7100 2075 7100 3175
 Wire Wire Line
 	7100 3175 7175 3175
 Wire Wire Line
-	5775 1575 7100 1575
+	5775 1575 6075 1575
+Wire Wire Line
+	6075 1575 7100 1575
 Wire Wire Line
 	6075 1575 6075 1650
@@
 Connection ~ 6075 1575
 Wire Wire Line
-	2550 1575 4975 1575
+	2550 1575 4525 1575
+Wire Wire Line
+	4525 1575 4900 1575
+Wire Wire Line
+	4900 1575 4975 1575
 Wire Wire Line
 	4975 1675 4900 1675
@@
 	5725 3425 5725 2900
 Wire Wire Line
-	5725 2900 4900 2900
+	5725 2900 5275 2900
+Wire Wire Line
+	5275 2900 4900 2900
 Wire Wire Line
 	5275 2900 5275 2950
 Wire Wire Line
-	4125 3525 7175 3525
-Wire Wire Line
-	3900 3775 7175 3775
+	4600 3525 7175 3525
+Wire Wire Line
+	3900 3775 5000 3775
+Wire Wire Line
+	5000 3775 7175 3775
 Wire Wire Line
 	4900 2900 4900 3000
@@
 	6025 5000 6025 4700
 Wire Wire Line
-	3750 3050 4125 3050
-Wire Wire Line
-	3000 3050 3450 3050
+	3750 3050 4425 3050
 Wire Wire Line
 	2375 3325 3900 3325
@@
 	6575 2675 6500 2675
 Wire Wire Line
-	2550 1425 2550 3025
+	2550 1425 2550 1575
+Wire Wire Line
+	2550 1575 2550 3025
 Wire Wire Line
 	2550 3025 2375 3025
@@
 	5950 2675 5950 3275
 Wire Wire Line
-	2375 2825 4425 2825
-Wire Wire Line
-	2375 2925 3000 2925
-Wire Wire Line
-	3000 2925 3000 3050
-Connection ~ 4125 3050
+	2375 2825 4600 2825
 Wire Wire Line
 	3450 3525 2375 3525
@@
 	2000 2500 2000 3275
 Wire Wire Line
-	4125 2525 4125 3625
-Wire Wire Line
-	4125 3625 2375 3625
-Connection ~ 4125 3525
-Wire Wire Line
-	7175 3625 4425 3625
-Wire Wire Line
-	4425 3625 4425 2825
+	2375 3625 4425 3625
+Wire Wire Line
+	4425 3625 7175 3625
+Wire Wire Line
+	2375 2925 3300 2925
+Wire Wire Line
+	3300 2925 3300 3050
+Wire Wire Line
+	3300 3050 3450 3050
+Wire Wire Line
+	4425 2675 4425 3050
+Wire Wire Line
+	4425 3050 4425 3625
+Connection ~ 4425 3625
+Wire Wire Line
+	4600 2825 4600 3525
+Connection ~ 4425 3050
+Text Label 3000 2825 0    50   ~ 0
+3.3V_TX
+$Comp
+L HEADER-MALE-1POS-TH-1x01 J2
+U 1 1 58AF2DFA
+P 2175 4475
+F 0 "J2" H 2125 4575 50  0000 L CNN
+F 1 "3.3V" H 2125 4375 50  0000 L CNN
+F 2 "Wickerlib:CONN-HEADER-STRAIGHT-P2.54MM-1x01" H 2175 4125 50  0001 C CIN
+F 3 "https://cdn.harwin.com/pdfs/60page140.pdf" H 2175 4475 5   0001 C CNN
+F 4 "HEADER MALE 1POS" H 2175 4125 50  0001 C CIN "Description"
+F 5 "Harwin" H 2175 4125 50  0001 C CIN "MF_Name"
+F 6 "M20-9992046" H 2175 4125 50  0001 C CIN "MF_PN"
+F 7 "Digikey" H 2175 4125 50  0001 C CIN "S1_Name"
+F 8 "952-1902-ND" H 2175 4125 50  0001 C CIN "S1_PN"
+	1    2175 4475
+	-1   0    0    -1
+$EndComp
+Wire Wire Line
+	2375 4475 2525 4475
+Wire Wire Line
+	2525 4475 2525 4425
+$Comp
+L +3.3V #PWR?
+U 1 1 58AF2F82
+P 2525 4425
+F 0 "#PWR?" H 2525 4275 50  0001 C CNN
+F 1 "+3.3V" H 2525 4565 50  0000 C CNN
+F 2 "" H 2525 4425 50  0000 C CNN
+F 3 "" H 2525 4425 50  0000 C CNN
+	1    2525 4425
+	1    0    0    -1
+$EndComp
 $EndSCHEMATC

Commit message: Fixed TX/RX.
Parts:
- removed D1: BAS16, Wickerlib:SOD-323, symbol DIODE-GEN-PURP-75V-250MA-BAS16-SOD323
- removed J2: 3.3V, Wickerlib:CONN-HEADER-STRAIGHT-P2.54MM-1x01, symbol HEADER-MALE-1POS-TH-1x01
- added D1: 1N4148, Wickerlib:SOD-123, symbol DIODE-GEN-PURP-75V-250MA-1N4148WTR-SOD123
Connections:
- net labels added: VCC
- net labels removed: +5V
- wire segments 73 -> 58
Other:
- note added: "To use with 5V FTDI:\nconnect FTDI cable\nstarting with RESET\n(green) at pin 1.\n\n\nTo use with 3.3V\ncontroller, connect\n to VCC, GPS_RX, \n3.3V_TX, and GND."
- note removed: "To use with 5V FTDI:\nconnect FTDI cable\nstarting with RESET\n(green) at pin 1.\n\n\nTo use with 3.3V\ncontroller, connect\n to 3.3V, GPS_RX, \n3.3V_TX, and GND."
- moved on the sheet: AN1, C2, R3

Commit message: Built and verified v1.1.
Parts:
- AN1: value UFL -> UFL GPS ANTENNA
Other:
- note added: "FGPMMOPA6H GPS Breakout Board v1.1"
Changed lines of the file:
@@
 EESchema Schematic File Version 2
+LIBS:fgpmmopa6h-gps-breakout-rescue
 LIBS:wickerlib
 LIBS:fgpmmopa6h-gps-breakout-cache
@@
 	1    0    0    -1
 $EndComp
-$Comp
-L CONN-UFL-HIROSE-R-SMD AN1
-U 1 1 5875EDAC
-P 7400 4700
-F 0 "AN1" H 7400 4825 50  0000 L CNN
-F 1 "UFL" H 7225 4600 50  0000 L CNN
-F 2 "Wickerlib:U.FL-COAX" H 7400 4350 50  0001 C CIN
-F 3 "http://media.digikey.com/pdf/Data%20Sheets/Hirose%20PDFs/UFL%20Series.pdf" H 7400 4700 3   0001 C CNN
-F 4 "Hirose" H 7400 4350 50  0001 C CIN "MF_Name"
-F 5 "U.FL-R-SMT-1(01)" H 7400 4350 50  0001 C CIN "MF_PN"
-F 6 "Digikey" H 7400 4350 50  0001 C CIN "S1_Name"
-F 7 "H122041-ND" H 7400 4350 50  0001 C CIN "S1_PN"
-F 8 "CONN UFL JACK STR 50 OHM SMD" H 7400 4350 50  0001 C CIN "Description"
-	1    7400 4700
-	1    0    0    -1
-$EndComp
-Text Notes 725  6450 0    100  ~ 0
+Text Notes 750  5975 0    100  ~ 0
 Based on Adafruit Ultimate GPS Breakout [1]\nand FGPMMOPA6H datasheet [2] reference circuits.\n\n[1] https://www.adafruit.com/products/790\n[2] https://cdn-shop.adafruit.com/datasheets/GlobalTop-FGPMMOPA6H-Datasheet-V0A.pdf
 Text Notes 1850 3575 2    50   ~ 0
@@
 	8250 3975 8350 3975
 Wire Wire Line
-	8350 3975 8350 4325
+	8350 3975 8350 4075
+Wire Wire Line
+	8350 4075 8350 4175
+Wire Wire Line
+	8350 4175 8350 4275
+Wire Wire Line
+	8350 4275 8350 4325
 Wire Wire Line
 	8250 4275 8350 4275
@@
 	5950 3275 7175 3275
 Wire Wire Line
-	7100 1400 7100 3175
+	7100 1400 7100 1575
+Wire Wire Line
+	7100 1575 7100 2075
+Wire Wire Line
+	7100 2075 7100 3175
 Wire Wire Line
 	7100 3175 7175 3175
 Wire Wire Line
-	5775 1575 7100 1575
+	5775 1575 6075 1575
+Wire Wire Line
+	6075 1575 7100 1575
 Wire Wire Line
 	6075 1575 6075 1650
@@
 Connection ~ 6075 1575
 Wire Wire Line
-	2550 1575 4975 1575
+	2550 1575 4525 1575
+Wire Wire Line
+	4525 1575 4900 1575
+Wire Wire Line
+	4900 1575 4975 1575
 Wire Wire Line
 	4975 1675 4900 1675
@@
 	7175 3425 5725 3425
 Wire Wire Line
-	5725 2900 5725 3425
-Wire Wire Line
-	4850 2900 5725 2900
+	5725 3425 5725 2900
+Wire Wire Line
+	5725 2900 5275 2900
+Wire Wire Line
+	5275 2900 4850 2900
 Wire Wire Line
 	5275 2900 5275 2950
@@
 	4600 3525 7175 3525
 Wire Wire Line
-	3900 3775 7175 3775
+	3900 3775 5000 3775
+Wire Wire Line
+	5000 3775 7175 3775
 Wire Wire Line
 	4850 2900 4850 3000
@@
 	6575 2675 6500 2675
 Wire Wire Line
-	2550 1425 2550 3025
+	2550 1525 2550 1575
+Wire Wire Line
+	2550 1575 2550 3025
 Wire Wire Line
 	2550 3025 2375 3025
@@
 	2000 2500 2000 3275
 Wire Wire Line
-	2375 3625 7175 3625
+	2375 3625 4425 3625
+Wire Wire Line
+	4425 3625 7175 3625
 Wire Wire Line
 	2375 2925 3375 2925
@@
 	3375 3050 3975 3050
 Wire Wire Line
-	4425 2675 4425 3625
+	4425 2675 4425 3050
+Wire Wire Line
+	4425 3050 4425 3625
 Connection ~ 4425 3625
 Wire Wire Line
@@
 L VCC #PWR014
 U 1 1 58B0216F
-P 2550 1425
-F 0 "#PWR014" H 2550 1275 50  0001 C CNN
-F 1 "VCC" H 2550 1565 50  0000 C CNN
-F 2 "" H 2550 1425 50  0000 C CNN
-F 3 "" H 2550 1425 50  0000 C CNN
-	1    2550 1425
-	1    0    0    -1
-$EndComp
+P 2550 1525
+F 0 "#PWR014" H 2550 1375 50  0001 C CNN
+F 1 "VCC" H 2550 1665 50  0000 C CNN
+F 2 "" H 2550 1525 50  0000 C CNN
+F 3 "" H 2550 1525 50  0000 C CNN
+	1    2550 1525
+	1    0    0    -1
+$EndComp
+$Comp
+L CONN-UFL-HIROSE-R-SMD AN1
+U 1 1 58C458F2
+P 7400 4700
+F 0 "AN1" H 7400 4825 50  0000 L CNN
+F 1 "UFL GPS ANTENNA" H 7500 4575 50  0000 L CNN
+F 2 "Wickerlib:U.FL-COAX" H 7400 4350 50  0001 C CIN
+F 3 "http://media.digikey.com/pdf/Data%20Sheets/Hirose%20PDFs/UFL%20Series.pdf" H 7400 4700 3   0001 C CNN
+F 4 "Hirose" H 7400 4350 50  0001 C CIN "MF_Name"
+F 5 "U.FL-R-SMT-1(01)" H 7400 4350 50  0001 C CIN "MF_PN"
+F 6 "Digikey" H 7400 4350 50  0001 C CIN "S1_Name"
+F 7 "H122041-ND" H 7400 4350 50  0001 C CIN "S1_PN"
+F 8 "CONN UFL JACK STR 50 OHM SMD" H 7400 4350 50  0001 C CIN "Description"
+	1    7400 4700
+	1    0    0    -1
+$EndComp
+Text Notes 775  1275 0    118  ~ 0
+FGPMMOPA6H GPS Breakout Board v1.1
 $EndSCHEMATC

Commit message: Regenerated bom and gerbers.
Other:
- note added: "WARNING: \n\nHand solder the GPS chip! \n\nWe had problems with 2D\nworking but the 3D fix \n(needed for faster speed \nreporting) not working after\nassembly in reflow oven."
- note removed: "FGPMMOPA6H GPS Breakout Board v1.1"
Changed lines of the file:
@@
 Text Label 3000 2925 0    50   ~ 0
 5V_RX
+Text Label 3000 2825 0    50   ~ 0
+3.3V_TX
+$Comp
+L DIODE-GEN-PURP-75V-250MA-1N4148WTR-SOD123 D1
+U 1 1 58AFEADD
+P 4150 3050
+F 0 "D1" V 4250 3025 50  0000 L CNN
+F 1 "1N4148" V 4025 3075 50  0000 C CNN
+F 2 "Wickerlib:SOD-123" H 4150 2700 50  0001 C CIN
+F 3 "http://www.vishay.com/docs/85752/bas16ws.pdf" V 4150 3075 5   0001 C CNN
+F 4 "DIODE GEN PURP 75V 250MA 1N4148 SOD123" H 4150 2700 50  0001 C CIN "Description"
+F 5 "SMC Diode" H 4150 2700 50  0001 C CIN "MF_Name"
+F 6 "1N4148WTR" H 4150 2700 50  0001 C CIN "MF_PN"
+F 7 "Digikey" H 4150 2700 50  0001 C CIN "S1_Name"
+F 8 "1655-1360-1-ND" H 4150 2700 50  0001 C CIN "S1_PN"
+	1    4150 3050
+	0    -1   -1   0
+$EndComp
+$Comp
+L VCC #PWR014
+U 1 1 58B0216F
+P 2550 1525
+F 0 "#PWR014" H 2550 1375 50  0001 C CNN
+F 1 "VCC" H 2550 1665 50  0000 C CNN
+F 2 "" H 2550 1525 50  0000 C CNN
+F 3 "" H 2550 1525 50  0000 C CNN
+	1    2550 1525
+	1    0    0    -1
+$EndComp
+$Comp
+L CONN-UFL-HIROSE-R-SMD AN1
+U 1 1 58C458F2
+P 7400 4700
+F 0 "AN1" H 7400 4825 50  0000 L CNN
+F 1 "UFL GPS ANTENNA" H 7500 4575 50  0000 L CNN
+F 2 "Wickerlib:U.FL-COAX" H 7400 4350 50  0001 C CIN
+F 3 "http://media.digikey.com/pdf/Data%20Sheets/Hirose%20PDFs/UFL%20Series.pdf" H 7400 4700 3   0001 C CNN
+F 4 "Hirose" H 7400 4350 50  0001 C CIN "MF_Name"
+F 5 "U.FL-R-SMT-1(01)" H 7400 4350 50  0001 C CIN "MF_PN"
+F 6 "Digikey" H 7400 4350 50  0001 C CIN "S1_Name"
+F 7 "H122041-ND" H 7400 4350 50  0001 C CIN "S1_PN"
+F 8 "CONN UFL JACK STR 50 OHM SMD" H 7400 4350 50  0001 C CIN "Description"
+	1    7400 4700
+	1    0    0    -1
+$EndComp
+Text Notes 7875 2775 0    100  ~ 0
+WARNING: \n\nHand solder the GPS chip! \n\nWe had problems with 2D\nworking but the 3D fix \n(needed for faster speed \nreporting) not working after\nassembly in reflow oven.
 Connection ~ 8350 4075
 Wire Wire Line
@@
 	8250 3975 8350 3975
 Wire Wire Line
-	8350 3975 8350 4075
-Wire Wire Line
-	8350 4075 8350 4175
-Wire Wire Line
-	8350 4175 8350 4275
-Wire Wire Line
-	8350 4275 8350 4325
+	8350 3975 8350 4325
 Wire Wire Line
 	8250 4275 8350 4275
@@
 	5950 3275 7175 3275
 Wire Wire Line
-	7100 1400 7100 1575
-Wire Wire Line
-	7100 1575 7100 2075
-Wire Wire Line
-	7100 2075 7100 3175
+	7100 1400 7100 3175
 Wire Wire Line
 	7100 3175 7175 3175
 Wire Wire Line
-	5775 1575 6075 1575
-Wire Wire Line
-	6075 1575 7100 1575
+	5775 1575 7100 1575
 Wire Wire Line
 	6075 1575 6075 1650
@@
 Connection ~ 6075 1575
 Wire Wire Line
-	2550 1575 4525 1575
-Wire Wire Line
-	4525 1575 4900 1575
-Wire Wire Line
-	4900 1575 4975 1575
+	2550 1575 4975 1575
 Wire Wire Line
 	4975 1675 4900 1675
@@
 	5725 3425 5725 2900
 Wire Wire Line
-	5725 2900 5275 2900
-Wire Wire Line
-	5275 2900 4850 2900
+	5725 2900 4850 2900
 Wire Wire Line
 	5275 2900 5275 2950
@@
 	4600 3525 7175 3525
 Wire Wire Line
-	3900 3775 5000 3775
-Wire Wire Line
-	5000 3775 7175 3775
+	3900 3775 7175 3775
 Wire Wire Line
 	4850 2900 4850 3000
@@
 	6575 2675 6500 2675
 Wire Wire Line
-	2550 1525 2550 1575
-Wire Wire Line
-	2550 1575 2550 3025
+	2550 1525 2550 3025
 Wire Wire Line
 	2550 3025 2375 3025
@@
 	2000 2500 2000 3275
 Wire Wire Line
-	2375 3625 4425 3625
-Wire Wire Line
-	4425 3625 7175 3625
+	2375 3625 7175 3625
 Wire Wire Line
 	2375 2925 3375 2925
@@
 	3375 3050 3975 3050
 Wire Wire Line
-	4425 2675 4425 3050
-Wire Wire Line
-	4425 3050 4425 3625
+	4425 2675 4425 3625
 Connection ~ 4425 3625
 Wire Wire Line
 	4600 2825 4600 3525
 Connection ~ 4425 3050
-Text Label 3000 2825 0    50   ~ 0
-3.3V_TX
-$Comp
-L DIODE-GEN-PURP-75V-250MA-1N4148WTR-SOD123 D1
-U 1 1 58AFEADD
-P 4150 3050
-F 0 "D1" V 4250 3025 50  0000 L CNN
-F 1 "1N4148" V 4025 3075 50  0000 C CNN
-F 2 "Wickerlib:SOD-123" H 4150 2700 50  0001 C CIN
-F 3 "http://www.vishay.com/docs/85752/bas16ws.pdf" V 4150 3075 5   0001 C CNN
-F 4 "DIODE GEN PURP 75V 250MA 1N4148 SOD123" H 4150 2700 50  0001 C CIN "Description"
-F 5 "SMC Diode" H 4150 2700 50  0001 C CIN "MF_Name"
-F 6 "1N4148WTR" H 4150 2700 50  0001 C CIN "MF_PN"
-F 7 "Digikey" H 4150 2700 50  0001 C CIN "S1_Name"
-F 8 "1655-1360-1-ND" H 4150 2700 50  0001 C CIN "S1_PN"
-	1    4150 3050
-	0    -1   -1   0
-$EndComp
-$Comp
-L VCC #PWR014
-U 1 1 58B0216F
-P 2550 1525
-F 0 "#PWR014" H 2550 1375 50  0001 C CNN
-F 1 "VCC" H 2550 1665 50  0000 C CNN
-F 2 "" H 2550 1525 50  0000 C CNN
-F 3 "" H 2550 1525 50  0000 C CNN
-	1    2550 1525
-	1    0    0    -1
-$EndComp
-$Comp
-L CONN-UFL-HIROSE-R-SMD AN1
-U 1 1 58C458F2
-P 7400 4700
-F 0 "AN1" H 7400 4825 50  0000 L CNN
-F 1 "UFL GPS ANTENNA" H 7500 4575 50  0000 L CNN
-F 2 "Wickerlib:U.FL-COAX" H 7400 4350 50  0001 C CIN
-F 3 "http://media.digikey.com/pdf/Data%20Sheets/Hirose%20PDFs/UFL%20Series.pdf" H 7400 4700 3   0001 C CNN
-F 4 "Hirose" H 7400 4350 50  0001 C CIN "MF_Name"
-F 5 "U.FL-R-SMT-1(01)" H 7400 4350 50  0001 C CIN "MF_PN"
-F 6 "Digikey" H 7400 4350 50  0001 C CIN "S1_Name"
-F 7 "H122041-ND" H 7400 4350 50  0001 C CIN "S1_PN"
-F 8 "CONN UFL JACK STR 50 OHM SMD" H 7400 4350 50  0001 C CIN "Description"
-	1    7400 4700
-	1    0    0    -1
-$EndComp
-Text Notes 775  1275 0    118  ~ 0
-FGPMMOPA6H GPS Breakout Board v1.1
+Wire Notes Line
+	9025 2950 8525 3350
+Wire Notes Line
+	8525 3350 8525 3175
+Wire Notes Line
+	8525 3350 8700 3350
 $EndSCHEMATC
