File: mcp73871-battery-mgmt-breakout/mcp73871-battery-mgmt-breakout.kicad_pcb (KiCad board)
At the start: 2 copper layers, 0 parts

Commit message: Release v1.0 MCP73871, needs ordered and tested.
Parts:
- added C1: 4.7uF, Wickerlib:RLC-1206-SMD, F.Cu at (119.2, 80.8)
- added C2: 4.7uF, Wickerlib:RLC-1206-SMD, F.Cu at (122.7, 86.8)
- added C3: 4.7uF, Wickerlib:RLC-1206-SMD, F.Cu at (132.1, 85.4)
- added J1: MICRO USB, Wickerlib:CONN-USB-MICRO-B-AMPHENOL-10118193-0001LF, F.Cu at (119.2, 75.4)
- added J2: JST PH, Wickerlib:CONN-JST-S2B-PH-SM4-TB, F.Cu at (130.3, 78.9)
- added J3: BREAKOUT1, Wickerlib:CONN-HEADER-STRAIGHT-P2.54MM-1x07, F.Cu at (116.8, 83.8)
- added J4: BREAKOUT2, Wickerlib:CONN-HEADER-STRAIGHT-P2.54MM-1x07, F.Cu at (139.7, 83.8)
- added LED1: AMBER, Wickerlib:LED-0603-SMD, F.Cu at (132.1, 93.4)
- added LED2: AMBER, Wickerlib:LED-0603-SMD, F.Cu at (132.1, 96.4)
- added LED3: AMBER, Wickerlib:LED-0603-SMD, F.Cu at (132.1, 99.5)
- added R1: 0 ohm, Wickerlib:RLC-0603-SMD, F.Cu at (122.8, 81.1)
- added R2: 470, Wickerlib:RLC-0603-SMD, F.Cu at (127.8, 93.3)
- added R3: 470, Wickerlib:RLC-0603-SMD, F.Cu at (127.7, 96.4)
- added R4: 470, Wickerlib:RLC-0603-SMD, F.Cu at (127.8, 99.6)
- added R5: NTC 10K, Wickerlib:RLC-0402-SMD, F.Cu at (123.9, 90.9)
- added R6: 2K, Wickerlib:RLC-0603-SMD, F.Cu at (132.4, 89.5)
- added R7: 100K, Wickerlib:RLC-0603-SMD, F.Cu at (130.5, 89.6)
- added REF**: SYMBOL-OSHW-LOGO-NOTEXT-SILK, Wickerlib:SYMBOL-OSHW-LOGO-NOTEXT-SILK, F.Cu at (138.7, 78.2)
- added U1: MCP73871, Wickerlib:QFN-20-1EP-4x4MM_P0.5MM, F.Cu at (126.8, 87.2)
Routing:
- net VUSB: track 0.00 -> 39.6 mm, vias 0 -> 3
- net GND: track 0.00 -> 36.5 mm, vias 0 -> 18
- net VBAT: track 0.00 -> 26.8 mm
- net /~PG: track 0.00 -> 20.1 mm
- net /STAT1: track 0.00 -> 19.1 mm, vias 0 -> 2
- net /STAT2: track 0.00 -> 18.9 mm, vias 0 -> 1
- net /PROG3: track 0.00 -> 16.6 mm
- net /CE: track 0.00 -> 16.2 mm, vias 0 -> 1
- net /~TE: track 0.00 -> 15.7 mm, vias 0 -> 2
- net VCC: track 0.00 -> 14.5 mm
- net /PROG1: track 0.00 -> 12.2 mm
- net /THERM: track 0.00 -> 11.3 mm
- net /PROG2: track 0.00 -> 10.1 mm
- net /SEL: track 0.00 -> 8.64 mm, vias 0 -> 1
- net Net-(C1-Pad1): track 0.00 -> 5.14 mm
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- added copper zone on B.Cu, net GND
- added copper zone on F.Cu, net GND
Other:
- board outline added: 27.9 x 27.9 mm
- net class Default: clearance 0.254 -> 0.01524
- rule trace_clearance: 0.1524 -> 0.01524
- board text added: "CE"
- board text added: "GND"
- board text added: "MCP73871 Battery Management Breakout v1.0"
- board text added: "PRG1"
- board text added: "PRG2"
- board text added: "PRG3"
- board text added: "SEL"
- board text added: "STAT1"
- board text added: "STAT2"
- board text added: "THRM"
- board text added: "VBAT"
- board text added: "VCC"
- board text added: "VUSB"
- board text added: "wickerbox.net"
- board text added: "~PG"
- board text added: "~TE"
