File: mcp73871-battery-mgmt-breakout/mcp73871-battery-mgmt-breakout.sch (KiCad schematic (older format))
At the start: 0 parts

Commit message: Initial schematic, connectors pending placement.
Parts:
- added B1: LIPO, Wickerlib:UNDEFINED, symbol BATT-LIPO-3.7V-500MAH-JST-2PIN
- added C1, C2, C3: 4.7uF, Wickerlib:RLC-1206-SMD, symbol CAP-CER-4.7UF-50V-X7R-1206
- added J1: MICRO USB, USB-10118193, symbol CONN-USB-MICRO-B-10118193
- added J2: JST PH, Wickerlib:CONN-JST-S2B-PH-SM4-TB, symbol HEADER-FEMALE-2POS-TH-1x02-JST-PH
- added J3: BREAKOUT1, Wickerlib:CONN-HEADER-STRAIGHT-P2.54MM-1x07, symbol HEADER-FEMALE-7POS-TH-1x07-P0.1IN
- added J4: BREAKOUT2, Wickerlib:CONN-HEADER-STRAIGHT-P2.54MM-1x07, symbol HEADER-FEMALE-7POS-TH-1x07-P0.1IN
- added LED1, LED2, LED3: AMBER, Wickerlib:LED-0603-SMD, symbol LED-AMBER-0603-SMT-L296-Q2R2
- added R1: 0 ohm, RLC-0603-SMD, symbol RES-0.0-JUMPER-1/8W-0603
- added R2, R3, R4: 470, RLC-0603-SMD, symbol RES-470-5%-1/4W-0603
- added R5: NTC 10K, Wickerlib:RLC-0402-SMD, symbol THERM-NTC-10K-1%-0402
- added R6: 2K, RLC-0603-SMD, symbol RES-2K-1%-1/8W-0603
- added R7: 100K, RLC-0603-SMD, symbol RES-100K-1%-1/10W-0603
- added U1: MCP73871, Wickerlib:QFN-20-1EP-4x4MM_P0.5MM, symbol IC-LI-ION-CONTROLLER-MCP73871-QFN20
Connections:
- new net: C1.1, J1.1 (VCC), R1.2
- new net: LED1.1 (K), R2.1
- new net: LED2.1 (K), R3.1
- new net: LED3.1 (K), R4.1
- new net CE: U1.17 (CE)
- new net GND: C1.2, C2.2, C3.2, J1.5 (GND), J2.2 (P2), R5.2, R6.2, R7.2, U1.10 (VSS), U1.11 (VSS), U1.21 (VSS)
- new net PROG1: R6.1, U1.13 (PROG1)
- new net PROG2: U1.4 (PROG2)
- new net PROG3: R7.1, U1.12 (PROG3)
- new net SEL: U1.3 (SEL)
- new net STAT1: R2.2, U1.8 (STAT1)
- new net STAT2: R3.2, U1.7 (STAT2)
- new net THERM: R5.1, U1.5 (THERM)
- new net VBAT: C3.1, J2.1 (P1), U1.14 (VBAT), U1.15 (VBAT), U1.16 (VBAT_SENSE)
- new net VCC: C2.1, U1.1 (OUT), U1.20 (OUT)
- new net VUSB: LED1.2 (A), LED2.2 (A), LED3.2 (A), R1.1, U1.18 (IN), U1.19 (IN), U1.2 (VPCC)
- new net ~PG: R4.2, U1.6 (~PG)
- new net ~TE: U1.9 (~TE)
- no-connect marks 0 -> 5
Other:
- note added: "VPCC DISABLED"

Commit message: Release v1.0 MCP73871, needs ordered and tested.
Parts:
- J1: footprint USB-10118193 -> Wickerlib:CONN-USB-MICRO-B-AMPHENOL-10118193-0001LF
- R1, R2, R3, R4, R6, R7: footprint RLC-0603-SMD -> Wickerlib:RLC-0603-SMD
Connections:
- net CE: now also J4.2 (P2)
- net GND: now also J4.7 (P7)
- net PROG1: now also J4.3 (P3)
- net PROG2: now also J3.4 (P4)
- net PROG3: now also J4.4 (P4)
- net SEL: now also J3.3 (P3)
- net STAT1: now also J4.6 (P6)
- net STAT2: now also J3.6 (P6)
- net THERM: now also J3.5 (P5)
- net VBAT: now also J4.1 (P1)
- net VCC: now also J3.2 (P2)
- net VUSB: now also J3.1 (P1)
- net ~PG: now also J3.7 (P7)
- net ~TE: now also J4.5 (P5)
Changed lines of the file:
@@
 F 0 "J1" H 1000 3300 50  0000 L CNN
 F 1 "MICRO USB" H 1000 2600 50  0000 L CNN
-F 2 "USB-10118193" H 1150 2600 50  0001 C CIN
+F 2 "Wickerlib:CONN-USB-MICRO-B-AMPHENOL-10118193-0001LF" H 1150 2600 50  0001 C CIN
 F 3 "http://portal.fciconnect.com/Comergent//fci/drawing/10118193.pdf" V 625 2975 5   0001 C CNN
 F 4 "USB MICRO-B RECEPTACLE 5PIN SMT R/A STUDS" H 1150 2600 50  0001 C CIN "Description"
@@
 F 0 "R2" H 2425 3300 50  0000 L CNN
 F 1 "470" H 2425 3200 50  0000 L CNN
-F 2 "RLC-0603-SMD" H 2375 2900 50  0001 C CIN
+F 2 "Wickerlib:RLC-0603-SMD" H 2375 2900 50  0001 C CIN
 F 3 "http://rohmfs.rohm.com/en/products/databook/datasheet/passive/resistor/chip_resistor/esr.pdf" H 2375 3250 5   0001 C CNN
 F 4 "RES SMD 470 OHM 5% 1/4W 0603" H 2375 2900 50  0001 C CIN "Description"
@@
 F 0 "R3" H 2875 3300 50  0000 L CNN
 F 1 "470" H 2875 3200 50  0000 L CNN
-F 2 "RLC-0603-SMD" H 2825 2900 50  0001 C CIN
+F 2 "Wickerlib:RLC-0603-SMD" H 2825 2900 50  0001 C CIN
 F 3 "http://rohmfs.rohm.com/en/products/databook/datasheet/passive/resistor/chip_resistor/esr.pdf" H 2825 3250 5   0001 C CNN
 F 4 "RES SMD 470 OHM 5% 1/4W 0603" H 2825 2900 50  0001 C CIN "Description"
@@
 F 0 "R4" H 3325 3300 50  0000 L CNN
 F 1 "470" H 3325 3200 50  0000 L CNN
-F 2 "RLC-0603-SMD" H 3275 2900 50  0001 C CIN
+F 2 "Wickerlib:RLC-0603-SMD" H 3275 2900 50  0001 C CIN
 F 3 "http://rohmfs.rohm.com/en/products/databook/datasheet/passive/resistor/chip_resistor/esr.pdf" H 3275 3250 5   0001 C CNN
 F 4 "RES SMD 470 OHM 5% 1/4W 0603" H 3275 2900 50  0001 C CIN "Description"
@@
 F 0 "R6" H 6225 3875 50  0000 L CNN
 F 1 "2K" H 6225 3775 50  0000 L CNN
-F 2 "RLC-0603-SMD" H 6175 3475 50  0001 C CIN
+F 2 "Wickerlib:RLC-0603-SMD" H 6175 3475 50  0001 C CIN
 F 3 "http://www.seielect.com/catalog/SEI-RNCP.pdf" H 6175 3825 5   0001 C CNN
 F 4 "RES SMD 2K OHM 1% 1/8W 0603" H 6175 3475 50  0001 C CIN "Description"
@@
 F 0 "R7" H 6550 3875 50  0000 L CNN
 F 1 "100K" H 6550 3775 50  0000 L CNN
-F 2 "RLC-0603-SMD" H 6500 3475 50  0001 C CIN
+F 2 "Wickerlib:RLC-0603-SMD" H 6500 3475 50  0001 C CIN
 F 3 "https://www.seielect.com/Catalog/SEI-RMCF_RMCP.pdf" H 6500 3825 5   0001 C CNN
 F 4 "RES SMD 100K OHM 1% 1/10W 0603" H 6500 3475 50  0001 C CIN "Description"
@@
 L GND #PWR014
 U 1 1 59721BB6
-P 7775 5575
-F 0 "#PWR014" H 7775 5325 50  0001 C CNN
-F 1 "GND" H 7775 5425 50  0000 C CNN
-F 2 "" H 7775 5575 50  0000 C CNN
-F 3 "" H 7775 5575 50  0000 C CNN
-	1    7775 5575
+P 7775 5475
+F 0 "#PWR014" H 7775 5225 50  0001 C CNN
+F 1 "GND" H 7775 5325 50  0000 C CNN
+F 2 "" H 7775 5475 50  0000 C CNN
+F 3 "" H 7775 5475 50  0000 C CNN
+	1    7775 5475
 	1    0    0    -1
 $EndComp
@@
 F 0 "R1" V 2025 2750 50  0000 C CNN
 F 1 "0 ohm" V 2175 2750 50  0000 C CNN
-F 2 "RLC-0603-SMD" H 2100 2400 50  0001 C CIN
+F 2 "Wickerlib:RLC-0603-SMD" H 2100 2400 50  0001 C CIN
 F 3 "http://www.vishay.com/docs/28705/mcx0x0xpro.pdf" H 2100 2750 5   0001 C CNN
 F 4 "RES SMD 0.0 OHM JUMPER 1/8W 0603" H 2100 2400 50  0001 C CIN "Description"
@@
 Wire Wire Line
 	7825 5275 6975 5275
-Wire Wire Line
-	6975 5375 7825 5375
 Entry Wire Line
 	6875 4675 6975 4775
@@
 Entry Wire Line
 	6875 5175 6975 5275
-Entry Wire Line
-	6875 5275 6975 5375
 NoConn ~ 1500 2850
 NoConn ~ 1500 2950
 NoConn ~ 1500 3050
+Text Label 7150 4875 0    50   ~ 0
+CE
+Text Label 7150 4050 0    50   ~ 0
+SEL
+Text Label 7150 4150 0    50   ~ 0
+PROG2
+Text Label 7150 5175 0    50   ~ 0
+~TE
+Text Label 7150 4975 0    50   ~ 0
+PROG1
+Text Label 7150 5075 0    50   ~ 0
+PROG3
+Text Label 7150 4250 0    50   ~ 0
+THERM
+Wire Wire Line
+	7775 5475 7775 5375
+Wire Wire Line
+	7225 3550 7225 3850
+Connection ~ 7225 3850
+Wire Wire Line
+	7475 3550 7475 4775
+Wire Wire Line
+	7775 5375 7825 5375
+Connection ~ 7475 4775
+Wire Wire Line
+	7725 3950 7725 3550
+Connection ~ 7725 3950
+Text Label 7150 4450 0    50   ~ 0
+~PG
+Text Label 7150 5275 0    50   ~ 0
+STAT1
+Text Label 7150 4350 0    50   ~ 0
+STAT2
 $EndSCHEMATC
