File: atsamd21g18-breakout/atsamd21g18-breakout.sch (KiCad schematic (older format))
At the start: 28 parts, among them J1 SWD, J2 MICRO USB, J3 HEADER-FEMALE-18POS-TH-1x18-P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, J4 HEADER-FEMALE-18POS-TH-1x18-P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, U1 BU33SD5WG 500mA, U2 IC-MCU-ATSAMD21G18A-TQFP48-CU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, X1 16MHz

Commit message: Saving unsaved file.
Parts:
- removed C5: 1uF, Wickerlib:RLC-0805-SMD, symbol CAP-CER-1UF-25V-X7R-0805
- added C5: 1uF, Wickerlib:RLC-0603-SMD, symbol CAP-CER-1UF-25V-X7R-0603
Connections:
- net GND: now also C5.2
- net at U2.43 (VDDCORE): now also C5.1
Changed lines of the file:
@@
 NoConn ~ 4525 4350
-$Comp
-L CAP-CER-1UF-25V-X7R-0805 C5
-U 1 1 59821455
-P 3800 4900
-F 0 "C5" H 3900 4950 50  0000 L CNN
-F 1 "1uF" H 3900 4850 50  0000 L CNN
-F 2 "Wickerlib:RLC-0805-SMD" H 3800 4550 50  0001 C CIN
-F 3 "http://www.samsungsem.com/kr/front/downloadcms.do?path=/kr/support/product-search/mlcc/__icsFiles/afieldfile/2014/11/05&fileName=C_CL21B104KACNNNC.pdf" H 3800 4900 5   0001 C CNN
-F 4 "CAP CER 1UF 25V X7R 0805" H 3800 4550 50  0001 C CIN "Description"
-F 5 "Samsung" H 3800 4550 50  0001 C CIN "MF_Name"
-F 6 "CL21B105KAFNNNE" H 3800 4550 50  0001 C CIN "MF_PN"
-F 7 "Digikey" H 3800 4550 50  0001 C CIN "S1_Name"
-F 8 "1276-1066-1-ND" H 3800 4550 50  0001 C CIN "S1_PN"
-	1    3800 4900
-	1    0    0    -1
-$EndComp
 $Comp
 L GND #PWR010
@@
 Text Label 7525 5325 0    50   ~ 0
 PB22
+$Comp
+L CAP-CER-1UF-25V-X7R-0603 C5
+U 1 1 598793E1
+P 3800 4900
+F 0 "C5" H 3875 4950 50  0000 L CNN
+F 1 "1uF" H 3875 4850 50  0000 L CNN
+F 2 "Wickerlib:RLC-0603-SMD" H 3800 4550 50  0001 C CIN
+F 3 "http://ds.yuden.co.jp/TYCOMPAS/ut/detail.do?productNo=TMK107B7105KA-T&fileName=TMK107B7105KA-T_SS&mode=specSheetDownload" H 3800 4900 5   0001 C CNN
+F 4 "CAP CER 1UF 25V X7R 0603" H 3800 4550 50  0001 C CIN "Description"
+F 5 "Taiyo Yuden" H 3800 4550 50  0001 C CIN "MF_Name"
+F 6 "TMK107B7105KA-T" H 3800 4550 50  0001 C CIN "MF_PN"
+F 7 "Digikey" H 3800 4550 50  0001 C CIN "S1_Name"
+F 8 "587-2984-1-ND" H 3800 4550 50  0001 C CIN "S1_PN"
+	1    3800 4900
+	1    0    0    -1
+$EndComp
 $EndSCHEMATC
